File: SCMv3.kicad_sch (KiCad schematic)
At the start: 183 parts, among them IC1 40106BPWR, IC2 40106BPWR, IC3 TL072, J1-CLK-IN1 PJ301M-12, J10-ROTATE1 PJ301M-12, J11-RST-SLP1 PJ301M-12, J2-OUT1 PJ301M-12, J3-OUT2 PJ301M-12, J4-OUT3 PJ301M-12, J5-OUT4 PJ301M-12, J6-OUT5 PJ301M-12, J7-OUT6 PJ301M-12, J8-OUT7 PJ301M-12, J9-OUT8 PJ301M-12, Q1 2N7002, Q2 2N7002, Q3 2N7002, Q4 2N7002, U1 ATMEGA328, U1 KA78L05, X1 16MHz

Commit message: combo schematic as of 6/21/21
Parts:
- added 7-OUT6, 8-OUT7, J2-OUT1, J3-OUT2, J4-OUT3, J5-OUT4, J6-OUT5, J9-OUT8: JACK-MONO-SWB, symbol clocker-12b-eagle-import:JACK-MONO-SWB
- added IC1 (x4), IC2 (x4): 40106, symbol 4xxx:40106
- added LED? (x8): RGB_CA_PLCC4, 4ms_LED:LED_PLCC-4, symbol 4ms_LED:RGB_CA_PLCC4
- added R? (x24): 4.7k_0603, 4ms_Resistor:R_0603, symbol 4ms_Resistor:4.7k_0603
- added R? (x8): 1k_0603, 4ms_Resistor:R_0603, symbol 4ms_Resistor:1k_0603
- added U?: ATmega328-A, Package_QFP:TQFP-32_7x7mm_P0.8mm, symbol MCU_Microchip_ATmega:ATmega328-A
Connections:
- net +VREF: now also LED?.2 (A), LED?.2 (A), LED?.2 (A), LED?.2 (A), LED?.2 (A), LED?.2 (A), LED?.2 (A), LED?.2 (A)
- net GND: now also 7-OUT6.GND (SLEEVE), 7-OUT6.P$2 (SLEEVE), 8-OUT7.GND (SLEEVE), 8-OUT7.P$2 (SLEEVE), J2-OUT1.GND (SLEEVE), J2-OUT1.P$2 (SLEEVE), J3-OUT2.GND (SLEEVE), J3-OUT2.P$2 (SLEEVE), J4-OUT3.GND (SLEEVE), J4-OUT3.P$2 (SLEEVE), J5-OUT4.GND (SLEEVE), J5-OUT4.P$2 (SLEEVE), J6-OUT5.GND (SLEEVE), J6-OUT5.P$2 (SLEEVE), J9-OUT8.GND (SLEEVE), J9-OUT8.P$2 (SLEEVE)
- new net: J4-OUT3.P$1 (TIP), R?.2
- new net: R?.1, R?.1, R?.1 (x8)
- new net: LED?.4 (CG), R?.2 (x8)
- new net: LED?.1 (CR), R?.2 (x8)
- new net: LED?.3 (CB), R?.2 (x8)
- new net: IC1.2, R?.1 (x4)
- new net: J3-OUT2.P$1 (TIP), R?.2
- new net: IC2.2, R?.1 (x4)
- new net: J6-OUT5.P$1 (TIP), R?.2
- new net: J9-OUT8.P$1 (TIP), R?.2
- new net: 8-OUT7.P$1 (TIP), R?.2
- new net: J2-OUT1.P$1 (TIP), R?.2
- new net: U?.21 (GND), U?.3 (GND), U?.5 (GND)
- new net: U?.4 (VCC), U?.6 (VCC)
- new net: 7-OUT6.P$1 (TIP), R?.2
- new net: J5-OUT4.P$1 (TIP), R?.2
Other:
- moved on the sheet: 'DUINO1, 5VSEL1, BREAKOUT1, C1, C10, C11, C2, C3, C4, C5, C6, C7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

Commit message: 6/21 scm  schematic
Parts:
- removed R? (x14): 4.7k_0603, 4ms_Resistor:R_0603, symbol 4ms_Resistor:4.7k_0603
- added C? (x2): 0.1uF_0603_16V, 4ms_Capacitor:C_0603, symbol 4ms_Capacitor:0.1uF_0603_16V
- added C? (x2): 9pF_0603_50V, 4ms_Capacitor:C_0603, symbol 4ms_Capacitor:9pF_0603_50V
- added C? (x3): 47uF_5x5.3_16V, 4ms_Capacitor:CP_Elec_5x5.3, symbol 4ms_Capacitor:47uF_5x5.3_16V
- added D? (x2): B140-E3, 4ms_Diode:D_SMA, symbol 4ms_Diode:B140-E3
- added IC3: TL082, 4ms_Package_SSOP:TSSOP-8_4.4x3mm_Pitch0.65mm, symbol 4ms_IC:TL082
- added unit 3 of IC3
- added unit 2 of IC3
- added J?: Conn_02x08, 4ms_Connector:Pins_2x08_2.54mm_TH, symbol 4ms_Connector:Conn_02x08
- added J? (x3): JACK-MONO-SWB, symbol clocker-12b-eagle-import:JACK-MONO-SWB
- added J?: Conn_01x02, 4ms_Connector:Pins_1x02_2.54mm_TH, symbol 4ms_Connector:Conn_01x02
- added J?: Conn_01x03, 4ms_Connector:Pins_1x03_2.54mm_TH_AudioInsRGndL, symbol 4ms_Connector:Conn_01x03
- added L?: FerriteBead_0603_1.5A, 4ms_Resistor:R_0603, symbol 4ms_Inductor:FerriteBead_0603_1.5A
- added R?: 10k_0603, 4ms_Resistor:R_0603, symbol 4ms_Resistor:10k_0603
- added R?: 470k_0603, 4ms_Resistor:R_0603, symbol 4ms_Resistor:470k_0603
- added TRIM?: TrimPot_T73YEt_10k, 4ms_Potentiometer:Pot_Trim_7x6.6mm_T73YE, symbol 4ms_Potentiometer:TrimPot_T73YEt_10k
- added VR1: MC78L05ACH, 4ms_Package_SOT:SOT89-3, symbol 4ms_Regulator:MC78L05ACH
- added VR2: 78L09, clocker-12b:SOT89, symbol clocker-12b-eagle-import:VREG-POS78R
- added Y?: 16MHz_18pF_FA238, 4ms_Crystal:FA-238, symbol 4ms_Crystal:16MHz_18pF_FA238
Connections:
- net +12V: now also C?.1, D?.1 (K), IC3.8 (V+), VR1.3 (IN), VR2.3 (IN)
- net +5V: now also C?.1, J?.2 (Pin_2), TRIM?.3 (Right)
- net +9V: now also C?.1, VR2.1 (OUT)
- net +VREF: no longer LED?.2 (A), LED?.2 (A), LED?.2 (A), LED?.2 (A), LED?.2 (A), LED?.2 (A), LED?.2 (A), LED?.2 (A)
- net -12V: now also D?.1 (K), J?.15 (-12V), J?.16 (P16)
- net GND: now also C?.2, C?.2, C?.2, C?.2, C?.2, C?.2, C?.2, J?.10 (GND), J?.11 (GND), J?.12 (GND), J?.13 (-12), J?.14 (-12V), J?.9 (GND), R?.2, R?.2, VR1.2 (GND), VR2.2A (GND), VR2.2B (GND)
- net IN-SW: now also IC3.6 (-), IC3.7
- net PB1: now reaches R?.1
- net PB1: now also IC1.3, U?.13 (PB1)
- net PD3: now reaches R?.1, R?.1, R?.1
- net PD3: now also U?.1 (PD3)
- net PB5: now reaches R?.1
- net PB5: now also IC2.13, U?.17 (PB5)
- net at R?.1: now also IC1.4; no longer IC1.2
- net at R?.1: now also IC2.12; no longer IC2.2
- net PB4: now reaches R?.1
- net PB4: now also IC2.11, U?.16 (PB4)
- net PB0: now reaches R?.1
- net PB0: now also IC1.1, U?.12 (PB0)
- net at R?.1: now also IC2.4; no longer IC2.2
- net PD6: now reaches R?.1
- net PD6: now also U?.10 (PD6)
- net PB3: now reaches R?.1
- net PB3: now also IC1.9, U?.15 (PB3)
- net PD7: now reaches U?.11 (PD7)
- net PB2: now reaches U?.14 (PB2)
- net PB2: now also IC1.5, R?.1
- net PD4: now reaches U?.2 (PD4)
- net PC0: now reaches U?.23 (PC0)
- net PC1: now reaches U?.24 (PC1)
- net PC2: now reaches U?.25 (PC2)
- net PC3: now reaches U?.26 (PC3)
- net PC4: now reaches U?.27 (PC4)
- net PC5: now reaches U?.28 (PC5)
- net PC6: now reaches U?.29 (~{RESET}/PC6)
- net PD0: now reaches U?.30 (PD0)
- net PD1: now reaches U?.31 (PD1)
- net PD2: now reaches U?.32 (PD2)
- net at U?.7 (XTAL1/PB6): now also C?.1, Y?.2
- net at U?.8 (XTAL2/PB7): now also C?.1, Y?.1
- net PD5: now reaches U?.9 (PD5)
- net at R?.1: now also IC2.10; no longer IC2.2
- net at R?.1: now also IC1.6; no longer IC1.2
- net at R?.1: now also IC1.8; no longer IC1.2
- new net: C?.1, D?.2 (A), IC3.4 (V-)
- new net: J?.1 (P1), J?.2 (P2), J?.2 (Pin_2)
- new net: J?.5 (+12V), J?.6 (P6), L?.1
- new net: D?.2 (A), J?.7 (12V), J?.8 (+12V)
- new net: R?.1, TRIM?.1 (Left)
- new net: IC3.5 (+), J?.1 (Pin_1), R?.1
- new net: IC3.3 (+), TRIM?.2 (Center)
- new net: J?.GND (SLEEVE), J?.P$2 (SLEEVE) (x3)
- new net: J?.1 (Pin_1), L?.2
- new net: C?.1, J?.3 (Pin_3), VR1.1 (OUT)
- new net VREF: IC3.1, IC3.2 (-), LED?.2 (A), LED?.2 (A), LED?.2 (A), LED?.2 (A), LED?.2 (A), LED?.2 (A), LED?.2 (A), LED?.2 (A)
- no-connect marks 5 -> 21
Other:
- note added: "40106 (IC1 AND IC2) Is generic part"
- note added: "Double check that VR1 is correct part"
- note added: "VR2 78L09 is generic"
- moved on the sheet: 5VSEL1, C10, C11, C6, C7, C8, D4, D5, H5A, H8A, IC3A, JP1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

Commit message: SCMV3 SCHEMATIC 6/21
Parts:
- removed J?: Conn_01x03, 4ms_Connector:Pins_1x03_2.54mm_TH_AudioInsRGndL, symbol 4ms_Connector:Conn_01x03
- removed L?: FerriteBead_0603_1.5A, 4ms_Resistor:R_0603, symbol 4ms_Inductor:FerriteBead_0603_1.5A
- removed VR1: MC78L05ACH, 4ms_Package_SOT:SOT89-3, symbol 4ms_Regulator:MC78L05ACH
- removed VR2: 78L09, clocker-12b:SOT89, symbol clocker-12b-eagle-import:VREG-POS78R
- added C? (x3): 330pF_0603_35V, 4ms_Capacitor:C_0603, symbol 4ms_Capacitor:330pF_0603_35V
- added C? (x6): 1nF_0603_50V, 4ms_Capacitor:C_0603, symbol 4ms_Capacitor:1nF_0603_50V
- added D? (x9): BAT54S, 4ms_Package_SOT:SOT23-3_PO132, symbol 4ms_Diode:BAT54S
- added unit 7 of IC1
- added unit 7 of IC2
- added unit 3 of IC2
- added IC? (x3): 40106, symbol 4xxx:40106
- added J?: JRESYNC, 4ms_Jack:EighthInch_PJ398SM, symbol 4ms_Jack:3.5mm_Mono_Switched_SymSmall_0.05
- added J?: JROTATE, 4ms_Jack:EighthInch_PJ398SM, symbol 4ms_Jack:3.5mm_Mono_Switched_SymSmall_0.05
- added J?: JPW, 4ms_Jack:EighthInch_PJ398SM, symbol 4ms_Jack:3.5mm_Mono_Switched_SymSmall_0.05
- added J?: JSHUFFLE, 4ms_Jack:EighthInch_PJ398SM, symbol 4ms_Jack:3.5mm_Mono_Switched_SymSmall_0.05
- added J?: JSLIP, 4ms_Jack:EighthInch_PJ398SM, symbol 4ms_Jack:3.5mm_Mono_Switched_SymSmall_0.05
- added J?: JSKIP, 4ms_Jack:EighthInch_PJ398SM, symbol 4ms_Jack:3.5mm_Mono_Switched_SymSmall_0.05
- added J?: ISP, 4ms_Connector:Pins_2x03_2.54mm_TH, symbol 4ms_Connector:Conn_02x03
- added JFAST, JMUTE: 3.5mm_Stereo_SymSmall_0.05, 4ms_Jack:EighthInch_PJ398SM, symbol 4ms_Jack:3.5mm_Mono_Switched_SymSmall_0.05
- added JRESYNC?: PJ301M-12, 4ms-main-parts:PJ301M-12-FIX, symbol SCMBO-rescue:JACK-MONO
- added LED?: BLUE, 4ms_LED:LED_PLCC-4, symbol 4ms_LED:RGB_CA_PLCC4
- added PPW_, PROTATE_, PSHUFFLE_, PSKIP_, PSLIP_, PSLIP_?: 9mm_NoDet_10k_DShaft, 4ms_Potentiometer:Pot_9mm_DShaft, symbol 4ms_Potentiometer:9mm_NoDet_10k_DShaft
- added Q? (x4): Si2318, Package_TO_SOT_SMD:SOT-23, symbol 4ms_Transistor:Si2318
- added R? (x10): 100k_0603, 4ms_Resistor:R_0603, symbol 4ms_Resistor:100k_0603
- added R? (x2): 470k_0603, 4ms_Resistor:R_0603, symbol 4ms_Resistor:470k_0603
- added R? (x11): 470R_0805_350mW, Resistor_SMD:R_0805_2012Metric, symbol 4ms_Resistor:470R_0805_350mW
- added R? (x3): 10k_0603, 4ms_Resistor:R_0603, symbol 4ms_Resistor:10k_0603
- added R?: 4.7k_0603, 4ms_Resistor:R_0603, symbol 4ms_Resistor:4.7k_0603
- added SW? (x2): Button_DPDT_Orange_Latching, 4ms_Switch:Button_LED_PB61303, symbol 4ms_Switch:Button_DPDT_Orange_Latching
- added VR1: L78M05CDT, 4ms_Package_TO:TO-252-2, symbol 4ms_Regulator:L78M05CDT
- added VR2: UA78L09, 4ms_Package_SOT:SOT89-3, symbol 4ms_Regulator:UA78L09
- 7-OUT6, 8-OUT7, J2-OUT1, J3-OUT2, J4-OUT3, J5-OUT4, J6-OUT5, J9-OUT8: footprint (none) -> 4ms_Jack:EighthInch_PJ398SM; symbol clocker-12b-eagle-import:JACK-MONO-SWB -> 4ms_Jack:3.5mm_Mono_Switched_SymSmall_0.05; Display (none) -> 3.5mm_Mono; Manufacturer (none) -> Wenzhou QingPu Electronics Co; Part Number (none) -> WQP-WQP518MA; Specifications (none) -> Audio 3.5mm Jack, mono, switched, PC-pin Vertical
- J?: value Conn_02x08 -> POWER
- J?: value JACK-MONO-SWB -> CLK-IN1; footprint (none) -> 4ms_Jack:EighthInch_PJ398SM; symbol clocker-12b-eagle-import:JACK-MONO-SWB -> 4ms_Jack:3.5mm_Mono_Switched_SymSmall_0.05; Display (none) -> 3.5mm_Mono; Manufacturer (none) -> Wenzhou QingPu Electronics Co; Part Number (none) -> WQP-WQP518MA; Specifications (none) -> Audio 3.5mm Jack, mono, switched, PC-pin Vertical
- J?: value JACK-MONO-SWB -> ROTATE1; footprint (none) -> 4ms_Jack:EighthInch_PJ398SM; symbol clocker-12b-eagle-import:JACK-MONO-SWB -> 4ms_Jack:3.5mm_Mono_Switched_SymSmall_0.05; Display (none) -> 3.5mm_Mono; Manufacturer (none) -> Wenzhou QingPu Electronics Co; Part Number (none) -> WQP-WQP518MA; Specifications (none) -> Audio 3.5mm Jack, mono, switched, PC-pin Vertical
- J?: value JACK-MONO-SWB -> SLP1; footprint (none) -> 4ms_Jack:EighthInch_PJ398SM; symbol clocker-12b-eagle-import:JACK-MONO-SWB -> 4ms_Jack:3.5mm_Mono_Switched_SymSmall_0.05; Display (none) -> 3.5mm_Mono; Manufacturer (none) -> Wenzhou QingPu Electronics Co; Part Number (none) -> WQP-WQP518MA; Specifications (none) -> Audio 3.5mm Jack, mono, switched, PC-pin Vertical
- LED? (x5): value RGB_CA_PLCC4 -> GREEN
- LED?: value RGB_CA_PLCC4 -> WHITE
- LED? (x2): value RGB_CA_PLCC4 -> BLUE
Connections:
- net CV2 is gone; now on net CV1: BREAKOUT1.2 (P$2), C5.1, D3.3 (COMMON), R3.2, U1.24 (P$24)
- net PB3 is gone; now on net MOSI: IC1.9, R?.1, U?.15 (PB3)
- net PB4 is gone; now on net MISO: IC2.11, R?.1, U?.16 (PB4)
- net PB5 is gone; now on net SCK: IC2.13, R?.1, U?.17 (PB5)
- net PD2 is gone; now on net CV1: U?.32 (PD2)
- net RESET is gone; now on net +5V: C9.2, ISP1.5 (P$5), R21.2, U1.29 (P$29)
- net +12V: now also Q?.3 (D), Q?.3 (D), R?.2, R?.2, VR1.1 (VI), VR2.3 (VI)
- net +5V: now also C?.1, U?.18 (AVCC), U?.20 (AREF), U?.4 (VCC), U?.6 (VCC), D?.2 (cathode), D?.2 (cathode), D?.2 (cathode), D?.2 (cathode), D?.2 (cathode), D?.2 (cathode), D?.2 (cathode), D?.2 (cathode), J?.2 (+12V), J?.3 (SW), J?.3 (SW), J?.5 (GND), PPW_.1 (Left), PSHUFFLE_.1 (Left), PSKIP_.1 (Left), R?.1, R?.2, VR1.3 (VO)
- net +9V: now also IC1.14 (VDD), IC2.14 (VDD), VR2.1 (VO)
- net CV1: now also C?.1, C?.1, C?.1, D?.3 (AK), D?.3 (AK), D?.3 (AK), R?.1, R?.2, R?.2, R?.2, R?.2
- net GND: now also 7-OUT6.2 (SHEILD), 8-OUT7.2 (SHEILD), J2-OUT1.2 (SHEILD), J3-OUT2.2 (SHEILD), J4-OUT3.2 (SHEILD), J5-OUT4.2 (SHEILD), J6-OUT5.2 (SHEILD), J9-OUT8.2 (SHEILD), J?.2 (SHEILD), J?.2 (SHEILD), J?.2 (SHEILD), U?.21 (GND), U?.3 (GND), U?.5 (GND), C?.2, C?.2, C?.2, C?.2, C?.2, C?.2, C?.2, C?.2, C?.2, D?.1 (Anode), D?.1 (Anode), D?.1 (Anode), D?.1 (Anode), D?.1 (Anode), D?.1 (Anode), D?.1 (Anode), IC1.7 (VSS), IC2.5, IC2.7 (VSS), IC?.11, IC?.13, IC?.9, J?.2 (SHEILD), J?.2 (SHEILD), J?.2 (SHEILD), J?.2 (SHEILD), J?.2 (SHEILD), J?.2 (SHEILD), J?.3 (SW), J?.6 (GND), JFAST.2 (SHEILD), JFAST.3 (SW), JMUTE.2 (SHEILD), JMUTE.3 (SW), PPW_.3 (Right), PPW_.4 (Tab1), PPW_.5 (Tab2), PROTATE_.1 (Left), PROTATE_.4 (Tab1), PROTATE_.5 (Tab2), PSHUFFLE_.3 (Right), PSHUFFLE_.4 (Tab1), PSHUFFLE_.5 (Tab2), PSKIP_.3 (Right), PSKIP_.4 (Tab1), PSKIP_.5 (Tab2), PSLIP_.4 (Tab1), PSLIP_.5 (Tab2), PSLIP_?.1 (Left), Q?.2 (S), Q?.2 (S), R?.1, R?.1, R?.1, R?.2, VR1.2 (GND), VR2.2 (GND); no longer 7-OUT6.GND (SLEEVE), 7-OUT6.P$2 (SLEEVE), 8-OUT7.GND (SLEEVE), 8-OUT7.P$2 (SLEEVE), J2-OUT1.GND (SLEEVE), J2-OUT1.P$2 (SLEEVE), J3-OUT2.GND (SLEEVE), J3-OUT2.P$2 (SLEEVE), J4-OUT3.GND (SLEEVE), J4-OUT3.P$2 (SLEEVE), J5-OUT4.GND (SLEEVE), J5-OUT4.P$2 (SLEEVE), J6-OUT5.GND (SLEEVE), J6-OUT5.P$2 (SLEEVE), J9-OUT8.GND (SLEEVE), J9-OUT8.P$2 (SLEEVE)
- net IN-SW: now also J?.3 (SW)
- net MISO: now also J?.1 (+12V)
- net MOSI: now also J?.4 (GND)
- net PD6: now also IC2.3, R?.1; no longer R?.1
- net PD7: now also IC2.1, R?.1
- net SCK: now also J?.3 (GND)
- net at R?.2: now also J4-OUT3.1 (SIG); no longer J4-OUT3.P$1 (TIP)
- net at J?.5 (+12V): no longer J?.6 (P6)
- net at R?.2: now also J3-OUT2.1 (SIG); no longer J3-OUT2.P$1 (TIP)
- net at R?.2: now also J6-OUT5.1 (SIG); no longer J6-OUT5.P$1 (TIP)
- net at R?.2: now also J9-OUT8.1 (SIG); no longer J9-OUT8.P$1 (TIP)
- net at R?.2: now also 8-OUT7.1 (SIG); no longer 8-OUT7.P$1 (TIP)
- net at R?.2: now also LED?.4 (CG); no longer LED?.3 (CB)
- net at R?.2: now also J2-OUT1.1 (SIG); no longer J2-OUT1.P$1 (TIP)
- net at R?.2: now also 7-OUT6.1 (SIG); no longer 7-OUT6.P$1 (TIP)
- net at R?.2: now also J5-OUT4.1 (SIG); no longer J5-OUT4.P$1 (TIP)
- net PC0 renamed PC0_ROTATE
- net PC1 renamed PC1_RESET
- net PC2 renamed PC2_PW
- net PC2_PW: now also C?.1, D?.3 (AK), R?.2, R?.2
- net PC3 renamed PC3_SKIP
- net PC3_SKIP: now also C?.1, D?.3 (AK), R?.2, R?.2
- net PC4 renamed PC4_SYNC
- net PC4_SYNC: now also C?.1, D?.3 (AK), R?.2
- net PC5 renamed PC5_SHUFFLE
- net PC5_SHUFFLE: now also C?.1, D?.3 (AK), R?.2, R?.2
- net PC6: no longer names the net of U?.29 (~{RESET}/PC6)
- net PC6: now also R?.1
- net PD4 renamed PD4_MUTE
- net PD4_MUTE: now also C?.1, D?.3 (AK), R?.1
- net PD5 renamed PD5_FAST
- net PD5_FAST: now also C?.1, D?.3 (AK), R?.1
- new net: PSHUFFLE_.2 (Center), R?.1
- new net: JMUTE.1 (SIG), R?.2, SW?.4 (UP-B)
- new net: PSKIP_.2 (Center), R?.1
- new net: Q?.1 (G), R?.1 (x4)
- new net: R?.2, SW?.5 (POLE-B) (x2)
- new net: R?.2, SW?.8 (C) (x2)
- new net: Q?.3 (D), R?.1, SW?.6 (DOWN-B) (x2)
- new net: R?.2, SW?.2 (POLE-A) (x2)
- new net: J?.1 (SIG), R?.1 (x6)
- new net: JFAST.1 (SIG), R?.2, SW?.4 (UP-B)
- new net: Q?.2 (S), SW?.7 (A) (x2)
- new net: PPW_.2 (Center), R?.1
- new net: PSLIP_?.2 (Center), R?.1
- new net: J?.1 (SIG), PSLIP_?.3 (Right)
- new net: J?.1 (SIG), PROTATE_.3 (Right)
- new net: J?.1 (SIG), R?.2, R?.2
- new net: PROTATE_.2 (Center), R?.1
- new net: LED?.3 (CB), R?.2
- new net SHUFFLE: J?.3 (SW), R?.1, R?.2
- no-connect marks 21 -> 47
Other:
- note added: "40106 (IC1 AND IC2) Is generic part Note to self- ask about which footprint to use when doing pcb"
- note added: "DELETE THIS SECTION BELOW? ITS FROM SCM. ROTATE AND SLIP JACKS THE JACKS ARE REDUNDANT, SEE THEIR COUNTERPARTS (FROM BO)AT THE RIGHT SIDE OF THE SCHEMATIC (NAMES JROTATE AND JSLIP)"
- note added: "PINS 5,6 AND 21 CAN BE FOUND ON THE PIN TABLE, BUT ARE HIDDEN ON THE FOOTPRINT. HOW DO WE GET THEM TO SHOW?"
- note removed: "40106 (IC1 AND IC2) Is generic part"
- note removed: "Double check that VR1 is correct part"
- note removed: "VR2 78L09 is generic"
- moved on the sheet: 5VSEL1, BFAST1, BMUTE1, BREAKOUT, C10, C11, C2, C3, C4, C5, C6, C7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

Commit message: SCM combo schematic 6/24
Parts:
- IC1, IC2, IC? (x3): footprint (none) -> 4ms_Package_SSOP:TSSOP-14_4.4x5mm_P0.65mm; symbol 4xxx:40106 -> 4ms_IC:CD40106BPWR; Display (none) -> 40106; Manufacturer (none) -> Texas Instruments; Manufacturer 2 (none) -> Texas Instruments; Part Number (none) -> CD40106BPWR; Part Number 2 (none) -> CD40106BPWR; Specifications (none) -> CMOS, Hex Inverting Schmitt Trigger, TSSOP-14
- U?: footprint Package_QFP:TQFP-32_7x7mm_P0.8mm -> 4ms_Package_QFP:TQFP-32_7x7mm_P0.8mm; symbol MCU_Microchip_ATmega:ATmega328-A -> 4ms_IC:ATMEGA328-AU; Display (none) -> ATMEGA328; Manufacturer (none) -> Microchip Technology / Atmel; Part Number (none) -> ATMEGA328-AU; Specifications (none) -> 8-bit Microcontrollers - MCU AVR 32K FLSH, 1K EE 2K SRAM - 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
Connections:
- net VREF: now also LED?.2 (A)
Other:
- note added: "DELETE THIS SECTION BELOW? ITS FROM SCM. ROTATE AND SLIP JACKS THE JACKS ARE REDUNDANT, SEE THEIR COUNTERPARTS (FROM BO)AT THE TOP RIGHT SIDE OF THE SCHEMATIC (NAMES JROTATE AND JSLIP)"
- note removed: "40106 (IC1 AND IC2) Is generic part Note to self- ask about which footprint to use when doing pcb"
- note removed: "DELETE THIS SECTION BELOW? ITS FROM SCM. ROTATE AND SLIP JACKS THE JACKS ARE REDUNDANT, SEE THEIR COUNTERPARTS (FROM BO)AT THE RIGHT SIDE OF THE SCHEMATIC (NAMES JROTATE AND JSLIP)"
- note removed: "PINS 5,6 AND 21 CAN BE FOUND ON THE PIN TABLE, BUT ARE HIDDEN ON THE FOOTPRINT. HOW DO WE GET THEM TO SHOW?"
- moved on the sheet: 7-OUT6, 8-OUT7, IC1G, IC2G, J2-OUT1, J3-OUT2, J4-OUT3, J5-OUT4, J6-OUT5, J9-OUT8, R?

Commit message: 6/25 SCM SCHEM
Parts:
- removed 'DUINO1: HEADER-1X6-TH, clocker-12b:HEADER-1X6-TH, symbol clocker-12b-eagle-import:HEADER-1X6
- removed 5VSEL1: HEADER-1X3-TH, clocker-12b:HEADER-1X3-TH, symbol clocker-12b-eagle-import:HEADER-1X3
- removed BFAST1, BMUTE1: ORANGE-LATCH, 4ms-footprints:BUTTON-LED-PB61303, symbol SCMBO-rescue:DPDT-ILLUM
- removed BREAKOUT: CONN_02X08, 4ms-footprints:HEADER-2X8-TH, symbol SCMBO-rescue:CONN_02X08
- removed BREAKOUT1: HEADER-2x8-SMT, clocker-12b:HEADER-2X8-SMT, symbol clocker-12b-eagle-import:HEADER-2X8BARE
- removed C1, C2: 9pF, clocker-12b:C0603, symbol clocker-12b-eagle-import:CB
- removed C1: 47uF, Capacitors_SMD:c_elec_5x5.3, symbol SCMBO-rescue:CP1_Small-Device
- removed C10, C11, C9: 0.1uF, clocker-12b:C0603, symbol clocker-12b-eagle-import:CB
- removed C2, C3, C4, C5, C6, C7: 1000pF, 4ms-footprints:C0603, symbol Device:C_Small
- removed C3, C4, C5: 330pF, clocker-12b:C0603, symbol clocker-12b-eagle-import:CB
- removed C6, C7, C8: 47uF, clocker-12b:C-POL-5, symbol clocker-12b-eagle-import:C-POL5
- removed C8: 0.1uF, 4ms-footprints:C0603, symbol Device:C_Small
- removed D1, D3, D4, D5, D6, D7: BAT54S, 4ms-footprints:SOT23, symbol SCMBO-rescue:D_Schottky_x2_Serial
- removed D1, D2, D3: BAT54S, clocker-12b:SOT23, symbol clocker-12b-eagle-import:DIODE-DUAL
- removed D2: B140, 4ms-footprints:SMA_Standard, symbol Device:D_Schottky
- removed D4, D5: B140-E3, clocker-12b:SMA, symbol clocker-12b-eagle-import:DA
- removed H4 (x6), H5 (x6), H6 (x6): HEADER-2X3-B2B-MALESMT, clocker-12b:HEADER-2X3-SMT, symbol clocker-12b-eagle-import:HEADER-2X3-B2B-MALESMT
- removed H7 (x6), H8 (x6), H9 (x6): HEADER-2X3-B2B-FEMALETH-BOT, clocker-12b:HEADER-2X3-TH-BOTTOM, symbol clocker-12b-eagle-import:HEADER-2X3-B2B-FEMALETH-BOT
- removed IC1 (x7), IC2 (x7): 40106BPWR, clocker-12b:TSSOP14, symbol clocker-12b-eagle-import:40106BPWR
- removed IC3 (x3): TL072, clocker-12b:SOIC8, symbol clocker-12b-eagle-import:OPAMP-2TL072M
- removed ISP1: HEADER-2X3-SMT, clocker-12b:HEADER-2X3-SMT, symbol clocker-12b-eagle-import:HEADER-2X3
- removed J1-CLK-IN1, J10-ROTATE1, J11-RST-SLP1, J2-OUT1, J3-OUT2, J4-OUT3, J5-OUT4, J6-OUT5, J7-OUT6, J8-OUT7, J9-OUT8: PJ301M-12, clocker-12b:PJ301M-12, symbol clocker-12b-eagle-import:JACK-MONO-SWM
- removed J?: ROTATE1, 4ms_Jack:EighthInch_PJ398SM, symbol 4ms_Jack:3.5mm_Mono_Switched_SymSmall_0.05
- removed J?: SLP1, 4ms_Jack:EighthInch_PJ398SM, symbol 4ms_Jack:3.5mm_Mono_Switched_SymSmall_0.05
- removed JFAST1, JMUTE1, JPW1, JRESYNC1, JRESYNC?, JROTATE1, JSHUFFLE1, JSKIP1, JSLIP1: PJ301M-12, 4ms-main-parts:PJ301M-12-FIX, symbol SCMBO-rescue:JACK-MONO
- removed JP1: 1x2-TH, clocker-12b:HEADER-1X2-TH, symbol clocker-12b-eagle-import:HEADER-1X2
- removed L1: BEAD, clocker-12b:0603, symbol clocker-12b-eagle-import:LB
- removed LED1: White, clocker-12b:LED-T1, symbol clocker-12b-eagle-import:LED
- removed LED2: Blue, clocker-12b:LED-T1, symbol clocker-12b-eagle-import:LED
- removed LED3, LED9: Red or blue, clocker-12b:LED-T1, symbol clocker-12b-eagle-import:LED
- removed LED4, LED7: Green, clocker-12b:LED-T1, symbol clocker-12b-eagle-import:LED
- removed LED5: Red or green, clocker-12b:LED-T1, symbol clocker-12b-eagle-import:LED
- removed LED6, LED8: Blue or green, clocker-12b:LED-T1, symbol clocker-12b-eagle-import:LED
- removed POWER1: HEADER-2X8-SMT, clocker-12b:HEADER-2X8-SMT-SHROUDED, symbol clocker-12b-eagle-import:HEADER-2X8SHRD
- removed PPW1, PSLIP1: 10k Center Det, 4ms-footprints:POT-9MM-ALPHA, symbol SCMBO-rescue:POT
- removed PROTATE1, PSHUFFLE1, PSKIP1: 10k No Det, 4ms-footprints:POT-9MM-ALPHA, symbol SCMBO-rescue:POT
- removed Q1, Q2, Q3, Q4: 2N7002, 4ms-footprints:SOT23, symbol Device:Q_NMOS_GSD
- removed R1, R11, R12, R13, R14, R16, R19, R4, R6, R8: 100k, 4ms-footprints:R0603, symbol Device:R
- removed R1, R2, R3: 470, clocker-12b:R0603, symbol clocker-12b-eagle-import:RB
- removed R10, R11, R4, R5, R6, R7, R8, R9: 1k, clocker-12b:R0603, symbol clocker-12b-eagle-import:RB
- removed R10, R15, R18, R2, R3, R5, R7: 470, 4ms-footprints:R0603, symbol Device:R
- removed R12, R13, R14, R15, R16, R17, R18, R19, R20, R21, R25: 10k, clocker-12b:R0603, symbol clocker-12b-eagle-import:RB
- removed R17, R9: 10k, 4ms-footprints:R0603, symbol Device:R
- removed R22, R23, R24, R26: 470k, clocker-12b:R0603, symbol clocker-12b-eagle-import:RB
- removed R? (x2): 470k_0603, 4ms_Resistor:R_0603, symbol 4ms_Resistor:470k_0603
- removed R? (x3): 470R_0805_350mW, Resistor_SMD:R_0805_2012Metric, symbol 4ms_Resistor:470R_0805_350mW
- removed RCD||SCM1: solder-blob, clocker-12b:SJ_2, symbol clocker-12b-eagle-import:SJ2W
- removed TR24: 10k, clocker-12b:PIHER-6MM, symbol clocker-12b-eagle-import:POT-MI
- removed U1: KA78L05, TO_SOT_Packages_SMD:SOT89-3_Housing, symbol SCMBO-rescue:MC78L05ACH
- removed U1: ATMEGA328, clocker-12b:TQFP-32, symbol clocker-12b-eagle-import:ATMEGA168
- removed VR1: 78M05, clocker-12b:DPAK, symbol clocker-12b-eagle-import:VREG-POS78A
- removed VR2: 78L09, clocker-12b:SOT89, symbol clocker-12b-eagle-import:VREG-POS78R
- removed X1: 16MHz, clocker-12b:FA-238, symbol clocker-12b-eagle-import:CRYSTALE
- R? (x8): footprint Resistor_SMD:R_0805_2012Metric -> 4ms_Resistor:R_0603; symbol 4ms_Resistor:470R_0805_350mW -> 4ms_Resistor:470R_0603; Display 470R/350mW -> 470R; JLCPCB ID (none) -> C23179; Manufacturer Panasonic -> Yageo; Part Number ERJ-P06J471V -> RC0603FR-07470RL; Specifications 470R, >=350mW, 5% -> 470R, 1%, 1/10W, 0603
Connections:
- net GND: now also D?.1 (Anode)
- net PC0_ROTATE: now also C?.1, D?.3 (AK), R?.2
- removed net CV1: C?.1, C?.1, C?.1, D?.3 (AK), D?.3 (AK), D?.3 (AK), R?.2, R?.2, R?.2, U?.32 (PD2)
- net PC1_RESET renamed PC1_SLIP
- net PC1_SLIP: now also C?.1, D?.3 (AK), R?.2
- new net PD2: C?.1, D?.3 (AK), R?.2, U?.32 (PD2)
- no-connect marks 47 -> 41
Other:
- note removed: "DELETE THIS SECTION BELOW? ITS FROM SCM. ROTATE AND SLIP JACKS THE JACKS ARE REDUNDANT, SEE THEIR COUNTERPARTS (FROM BO)AT THE TOP RIGHT SIDE OF THE SCHEMATIC (NAMES JROTATE AND JSLIP)"
- note removed: "MUTE"
- note removed: "NC"
- note removed: "PW"
- note removed: "RESYNC"
- note removed: "ROT"
- note removed: "SHUFFLE"
- note removed: "SKIP"
- note removed: "SLIP"
- note removed: "SNIP H2 PINS 1-4 FOR RCD"
- note removed: "x4"
- moved on the sheet: C?, D?, J?, PROTATE_A, PROTATE_B, PSLIP_?A, PSLIP_B, R?
