File: SCMv3.kicad_sch (KiCad schematic)
At the start: 121 parts, among them IC1 40106, IC2 40106, IC3 TL082, J2-OUT1 JACK-MONO-SWB, J3-OUT2 JACK-MONO-SWB, J4-OUT3 JACK-MONO-SWB, J5-OUT4 JACK-MONO-SWB, J6-OUT5 JACK-MONO-SWB, J9-OUT8 JACK-MONO-SWB

Commit message: SCHEM + PCB 6/
Parts:
- PPW1: renamed from PPW_; value 9mm_NoDet_10k_DShaft -> 9mm_CtrDet_10k_DShaft; footprint 4ms_Potentiometer:Pot_9mm_DShaft -> 4ms_Potentiometer:Pot_9mm_Dshaft_Det; symbol 4ms_Potentiometer:9mm_NoDet_10k_DShaft -> 4ms_Potentiometer:9mm_CtrDet_10k_DShaft; Part Number RV09BCF-40-25F-B10K-007 -> RV09BCF-40-25F-B10K-0C7; Specifications 10k Linear, 9mm pot, No Detent, D-Shaft -> 10k Linear, 9mm pot, Center Detent, D-Shaft
- PROTATE1: renamed from PROTATE_; value 9mm_NoDet_10k_DShaft -> 9mm_CtrDet_10k_DShaft; footprint 4ms_Potentiometer:Pot_9mm_DShaft -> 4ms_Potentiometer:Pot_9mm_Dshaft_Det; symbol 4ms_Potentiometer:9mm_NoDet_10k_DShaft -> 4ms_Potentiometer:9mm_CtrDet_10k_DShaft; Part Number RV09BCF-40-25F-B10K-007 -> RV09BCF-40-25F-B10K-0C7; Specifications 10k Linear, 9mm pot, No Detent, D-Shaft -> 10k Linear, 9mm pot, Center Detent, D-Shaft
- PSHUFFLE1: renamed from PSHUFFLE_; value 9mm_NoDet_10k_DShaft -> 9mm_CtrDet_10k_DShaft; footprint 4ms_Potentiometer:Pot_9mm_DShaft -> 4ms_Potentiometer:Pot_9mm_Dshaft_Det; symbol 4ms_Potentiometer:9mm_NoDet_10k_DShaft -> 4ms_Potentiometer:9mm_CtrDet_10k_DShaft; Part Number RV09BCF-40-25F-B10K-007 -> RV09BCF-40-25F-B10K-0C7; Specifications 10k Linear, 9mm pot, No Detent, D-Shaft -> 10k Linear, 9mm pot, Center Detent, D-Shaft
- PSKIP1: renamed from PSKIP_; value 9mm_NoDet_10k_DShaft -> 9mm_CtrDet_10k_DShaft; footprint 4ms_Potentiometer:Pot_9mm_DShaft -> 4ms_Potentiometer:Pot_9mm_Dshaft_Det; symbol 4ms_Potentiometer:9mm_NoDet_10k_DShaft -> 4ms_Potentiometer:9mm_CtrDet_10k_DShaft; Part Number RV09BCF-40-25F-B10K-007 -> RV09BCF-40-25F-B10K-0C7; Specifications 10k Linear, 9mm pot, No Detent, D-Shaft -> 10k Linear, 9mm pot, Center Detent, D-Shaft
- PSLIP1: renamed from PSLIP_?; value 9mm_NoDet_10k_DShaft -> 9mm_CtrDet_10k_DShaft; footprint 4ms_Potentiometer:Pot_9mm_DShaft -> 4ms_Potentiometer:Pot_9mm_Dshaft_Det; symbol 4ms_Potentiometer:9mm_NoDet_10k_DShaft -> 4ms_Potentiometer:9mm_CtrDet_10k_DShaft; Part Number RV09BCF-40-25F-B10K-007 -> RV09BCF-40-25F-B10K-0C7; Specifications 10k Linear, 9mm pot, No Detent, D-Shaft -> 10k Linear, 9mm pot, Center Detent, D-Shaft
- PSLIP1: renamed from PSLIP_; value 9mm_NoDet_10k_DShaft -> 9mm_CtrDet_10k_DShaft; footprint 4ms_Potentiometer:Pot_9mm_DShaft -> 4ms_Potentiometer:Pot_9mm_Dshaft_Det; symbol 4ms_Potentiometer:9mm_NoDet_10k_DShaft -> 4ms_Potentiometer:9mm_CtrDet_10k_DShaft; Part Number RV09BCF-40-25F-B10K-007 -> RV09BCF-40-25F-B10K-0C7; Specifications 10k Linear, 9mm pot, No Detent, D-Shaft -> 10k Linear, 9mm pot, Center Detent, D-Shaft
- gave numbers to parts that had none: 18
- renumbered J9-OUT8 to J1-OUT8, 8-OUT7 to J2-OUT7, 7-OUT6 to J3-OUT6, J6-OUT5 to J4-OUT5, J4-OUT3 to J6-OUT3, J3-OUT2 to J7-OUT2, J2-OUT1 to J8-OUT1, JFAST to JFAST1, JMUTE to JMUTE1
Connections:
- net MISO renamed UC_OUT5_MISO
- net MOSI renamed UC_OUT4_MOSI
- net PB0 renamed UC_OUT1
- net PB1 renamed UC_OUT2
- net PB2 renamed UC_OUT3
- net PC0_ROTATE renamed UC_ROTATE
- net PC1_SLIP renamed UC_SLIP
- net PC2_PW renamed UC_PW
- net PC3_SKIP renamed UC_SKIP
- net PC4_SYNC renamed UC_SYNC
- net PC5_SHUFFLE renamed UC_SHUFFLE
- net PD0: no longer names the net of U?.30 (PD0)
- net PD1: no longer names the net of U?.31 (PD1)
- net PD2 renamed UC_CLK_IN
- net PD3 renamed UC_IN
- net PD4_MUTE renamed UC_MUTE
- net PD5_FAST renamed UC_FAST
- net PD6 renamed UC_OUT8
- net PD7 renamed UC_OUT7
- net SCK renamed UC_OUT6_SCK
- no-connect marks 41 -> 43

Commit message: PCB + SCHEM 6/30
Parts:
- J9-CLK_IN1: renamed from J9-CLK_IN; value CLK-IN1 -> JCLK_IN
- gave numbers to parts that had none: 80
- renumbered IC2 to IC1
Connections:
- net +5V: now also D7.2 (cathode)
- net GND: now also D5.1 (Anode)

Commit message: PCB +SCHEM 7/02
Parts:
- added C17, C18, C19, C20, C21: 0.1uF_0603_16V, 4ms_Capacitor:C_0603, symbol 4ms_Capacitor:0.1uF_0603_16V
Connections:
- net +12V: now also C19.1
- net +9V: now also C17.1, C20.1
- net GND: now also C17.2, C18.2, C19.2, C20.2, C21.2; no longer IC1.7 (VSS), IC2.7 (VSS)
- net -12VA: now reaches C16.1, D11.2 (A), IC3.4 (V-)
- net -12V: no longer names the net of D11.1 (K), J3.15 (-12V), J3.16 (P16)
- new net: C21.1, IC2.7 (VSS)
- new net: C18.1, IC1.7 (VSS)
Other:
- moved on the sheet: C15, IC1G, IC2G

Commit message: Fixes/tweaks to sch+pcb:
-Changed PCB form 16-layer to 2-layer board.
-RESET net was attached to +5V, moved it to _RESET/PC6 pin 29 of U1
-Renamed net UC_IN to UC_LED_IN (it only drives the IN LED, nothing else)
Connections:
- net +5V: no longer J1.5 (GND)
- net RESET: now reaches R16.1, U1.29 (~{RESET}/PC6)
- net RESET: now also J1.5 (GND)
- net UC_IN renamed UC_LED_IN
Changed lines of the file:
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@@
-(kicad_sch (version 20210615) (generator eeschema)
+(kicad_sch (version 20210621) (generator eeschema)
   (paper "A2")
   (junction (at 35.56 331.47) (diameter 1.016) (color 0 0 0 0))
@@
   (junction (at 88.9 128.27) (diameter 1.016) (color 0 0 0 0))
   (junction (at 102.87 351.79) (diameter 1.016) (color 0 0 0 0))
+  (junction (at 107.95 97.79) (diameter 1.016) (color 0 0 0 0))
   (junction (at 118.11 327.66) (diameter 1.016) (color 0 0 0 0))
-  (junction (at 125.73 97.79) (diameter 1.016) (color 0 0 0 0))
   (junction (at 133.35 77.47) (diameter 1.016) (color 0 0 0 0))
   (junction (at 143.51 77.47) (diameter 1.016) (color 0 0 0 0))
@@
     (stroke (width 0) (type solid) (color 0 0 0 0))
   )
-  (wire (pts (xy 104.14 97.79) (xy 116.84 97.79))
+  (wire (pts (xy 104.14 97.79) (xy 107.95 97.79))
     (stroke (width 0) (type solid) (color 0 0 0 0))
   )
@@
     (stroke (width 0) (type solid) (color 0 0 0 0))
   )
+  (wire (pts (xy 107.95 97.79) (xy 116.84 97.79))
+    (stroke (width 0) (type solid) (color 0 0 0 0))
+  )
+  (wire (pts (xy 107.95 101.6) (xy 107.95 97.79))
+    (stroke (width 0) (type solid) (color 0 0 0 0))
+  )
+  (wire (pts (xy 109.22 101.6) (xy 107.95 101.6))
+    (stroke (width 0) (type solid) (color 0 0 0 0))
+  )
   (wire (pts (xy 115.57 327.66) (xy 118.11 327.66))
     (stroke (width 0) (type solid) (color 0 0 0 0))
@@
     (stroke (width 0) (type solid) (color 0 0 0 0))
   )
-  (wire (pts (xy 124.46 97.79) (xy 125.73 97.79))
-    (stroke (width 0) (type solid) (color 0 0 0 0))
-  )
-  (wire (pts (xy 125.73 97.79) (xy 127 97.79))
-    (stroke (width 0) (type solid) (color 0 0 0 0))
-  )
-  (wire (pts (xy 125.73 101.6) (xy 125.73 97.79))
-    (stroke (width 0) (type solid) (color 0 0 0 0))
-  )
-  (wire (pts (xy 127 101.6) (xy 125.73 101.6))
+  (wire (pts (xy 124.46 97.79) (xy 127 97.79))
     (stroke (width 0) (type solid) (color 0 0 0 0))
   )
@@
     (effects (font (size 1.27 1.27)) (justify left bottom))
   )
-  (label "UC_IN" (at 104.14 110.49 0)
+  (label "UC_LED_IN" (at 104.14 110.49 0)
     (effects (font (size 1.27 1.27)) (justify left bottom))
   )
@@
     (effects (font (size 1.27 1.27)) (justify left bottom))
   )
-  (label "RESET" (at 127 101.6 0)
-    (effects (font (size 1.27 1.27)) (justify left bottom))
-  )
-  (label "UC_IN" (at 171.45 31.75 180)
+  (label "RESET" (at 109.22 101.6 0)
+    (effects (font (size 1.27 1.27)) (justify left bottom))
+  )
+  (label "UC_LED_IN" (at 171.45 31.75 180)
     (effects (font (size 1.27 1.27)) (justify right bottom))
   )
