File: p2/SCMv3.kicad_sch (KiCad schematic)
At the start: 122 parts, among them IC1 40106, IC2 40106, IC3 TL082, J1 ISP, J1-OUT8 JACK-MONO-SWB, J2 Conn_01x02, J2-OUT7 JACK-MONO-SWB, J3 POWER, J3-OUT6 JACK-MONO-SWB, J4-OUT5 JACK-MONO-SWB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

Commit message: Restored p2
Parts:
- removed J?: Conn_01x02, 4ms_Connector:Pins_1x02_2.54mm_TH, symbol 4ms_Connector:Conn_01x02
- removed U?: STM32F030K6Tx, Package_QFP:LQFP-32_7x7mm_P0.8mm, symbol MCU_ST_STM32F0:STM32F030K6Tx
Connections:
- net +8V renamed +9V
