File: p3/SCMv3.kicad_sch (KiCad schematic)
At the start: 126 parts, among them IC1 40106, IC2 40106, IC3 TL082, J1 Conn_01x06, J1-OUT8 JACK-MONO-SWB, J2 Conn_01x02, J2-OUT7 JACK-MONO-SWB, J3 POWER, J3-OUT6 JACK-MONO-SWB, J4 Conn_01x02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

Commit message: Revert "Merge remote-tracking branch 'origin/main' into main"
This reverts commit 63f0bb0c0b25969e804c40226811b6ef72d39a13.
Connections:
- net SWCLK: now also U1.23 (PA13); no longer U1.24 (PA14)
- net SWDIO: now also U1.22 (PA12); no longer U1.23 (PA13)
- net UC_CLK_IN: now also U1.24 (PA14); no longer U1.22 (PA12)
