File: p5/SCMplus.kicad_sch (KiCad schematic)
At the start: 143 parts, among them J1 Conn_01x06, J1-OUT8 3.5mm_Mono_Switched_SymSmall_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, J2 Conn_01x02, J2-OUT7 3.5mm_Mono_Switched_SymSmall_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, J3 Conn_02x08, J3-OUT6 3.5mm_Mono_Switched_SymSmall_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, J4 Conn_01x02, J4-OUT5 3.5mm_Mono_Switched_SymSmall_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, J5-OUT4 3.5mm_Mono_Switched_SymSmall_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, J6-OUT3 3.5mm_Mono_Switched_SymSmall_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

Commit message: p5 BOM, gerbers, pos. Submitted for quote from Posin
Parts:
- C12, C15, C16, C17, C18, C19, C20, C23, C24, C25, C26, C27, C28, C29, C30: Manufacturer (none) -> AVX Corporation; Part Number (none) -> 0603YC104KAT2A
- C13, C14: Part Number VE-470M1CTR-0505 -> VES470M1CTR-0505
- C22: value 0.1uF_0603_16V -> 100nF_0603_16V; symbol 4ms_Capacitor:0.1uF_0603_16V -> 4ms_Capacitor:100nF_0603_16V; JLCPCB ID (none) -> C14663; Manufacturer (none) -> AVX Corporation; Part Number (none) -> 0603YC104KAT2A
- PPW1, PROTATE1, PSHUFFLE1, PSKIP1, PSLIP1: Manufacturer Song Huei -> Song Huei; Part Number RV16AF-4A-15FW-B100K-3 -> R0904N-B100K L-25KQ/LWS

Commit message: EQ from Posin, fixed many BOM errors on BOM and schematic
Parts:
- R16, R44, R45, R47, R48, R50: value 100k_0603 -> 10k_0603
- R22: value 4.7k_0603 -> 10k_0603
- R3, R36, R7: value 470R_0603 -> 10k_0603
- R30, R37, R39: value 100k_0603 -> 15k_0603
- R43, R46, R49: value 100R_0603 -> 1k_0603
Changed lines of the file:
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@@
     (in_bom yes) (on_board yes) (fields_autoplaced)
     (property "Reference" "R46" (id 0) (at 480.06 210.82 90))
-    (property "Value" "100R_0603" (id 1) (at 480.06 219.71 90)
+    (property "Value" "1k_0603" (id 1) (at 480.06 219.71 90)
       (effects (font (size 1.27 1.27)) hide)
     )
@@
     (in_bom yes) (on_board yes) (fields_autoplaced)
     (property "Reference" "R37" (id 0) (at 386.08 226.4242 90))
-    (property "Value" "100k_0603" (id 1) (at 386.08 233.68 90)
+    (property "Value" "15k_0603" (id 1) (at 386.08 233.68 90)
       (effects (font (size 1.27 1.27)) hide)
     )
@@
     (in_bom yes) (on_board yes) (fields_autoplaced)
     (property "Reference" "R43" (id 0) (at 480.06 153.67 90))
-    (property "Value" "100R_0603" (id 1) (at 480.06 162.56 90)
+    (property "Value" "1k_0603" (id 1) (at 480.06 162.56 90)
       (effects (font (size 1.27 1.27)) hide)
     )
@@
     (in_bom yes) (on_board yes) (fields_autoplaced)
     (property "Reference" "R7" (id 0) (at 274.32 297.5442 90))
-    (property "Value" "470R_0603" (id 1) (at 274.32 304.8 90)
+    (property "Value" "10k_0603" (id 1) (at 274.32 304.8 90)
       (effects (font (size 1.27 1.27)) hide)
     )
@@
     (in_bom yes) (on_board yes) (fields_autoplaced)
     (property "Reference" "R3" (id 0) (at 389.89 339.4542 90))
-    (property "Value" "470R_0603" (id 1) (at 389.89 346.71 90)
+    (property "Value" "10k_0603" (id 1) (at 389.89 346.71 90)
       (effects (font (size 1.27 1.27)) hide)
     )
@@
     (in_bom yes) (on_board yes) (fields_autoplaced)
     (property "Reference" "R48" (id 0) (at 426.72 272.1442 90))
-    (property "Value" "100k_0603" (id 1) (at 426.72 279.4 90)
+    (property "Value" "10k_0603" (id 1) (at 426.72 279.4 90)
       (effects (font (size 1.27 1.27)) hide)
     )
@@
     (in_bom yes) (on_board yes) (fields_autoplaced)
     (property "Reference" "R45" (id 0) (at 426.72 209.9142 90))
-    (property "Value" "100k_0603" (id 1) (at 426.72 217.17 90)
+    (property "Value" "10k_0603" (id 1) (at 426.72 217.17 90)
       (effects (font (size 1.27 1.27)) hide)
     )
@@
     (in_bom yes) (on_board yes) (fields_autoplaced)
     (property "Reference" "R22" (id 0) (at 273.05 367.3942 90))
-    (property "Value" "4.7k_0603" (id 1) (at 273.05 374.65 90)
+    (property "Value" "10k_0603" (id 1) (at 273.05 374.65 90)
       (effects (font (size 1.27 1.27)) hide)
     )
@@
     (in_bom yes) (on_board yes) (fields_autoplaced)
     (property "Reference" "R30" (id 0) (at 386.08 167.64 90))
-    (property "Value" "100k_0603" (id 1) (at 386.08 176.53 90)
+    (property "Value" "15k_0603" (id 1) (at 386.08 176.53 90)
       (effects (font (size 1.27 1.27)) hide)
     )
@@
     (in_bom yes) (on_board yes) (fields_autoplaced)
     (property "Reference" "R16" (id 0) (at 426.72 152.7642 90))
-    (property "Value" "100k_0603" (id 1) (at 426.72 160.02 90)
+    (property "Value" "10k_0603" (id 1) (at 426.72 160.02 90)
       (effects (font (size 1.27 1.27)) hide)
     )
@@
       (effects (font (size 1.27 1.27)) (justify left) hide)
     )
-    (property "Part Number" "0603YC104KAT2A" (id 7) (at 118.11 391.922 0)
+    (property "Part Number" "0603YC104KAT2A" (id 8) (at 118.11 391.922 0)
       (effects (font (size 1.27 1.27)) (justify left) hide)
     )
@@
     (in_bom yes) (on_board yes) (fields_autoplaced)
     (property "Reference" "R44" (id 0) (at 405.13 169.2742 90))
-    (property "Value" "100k_0603" (id 1) (at 405.13 176.53 90)
+    (property "Value" "10k_0603" (id 1) (at 405.13 176.53 90)
       (effects (font (size 1.27 1.27)) hide)
     )
@@
     (in_bom yes) (on_board yes) (fields_autoplaced)
     (property "Reference" "R49" (id 0) (at 480.06 273.05 90))
-    (property "Value" "100R_0603" (id 1) (at 480.06 281.94 90)
+    (property "Value" "1k_0603" (id 1) (at 480.06 281.94 90)
       (effects (font (size 1.27 1.27)) hide)
     )
@@
     (in_bom yes) (on_board yes) (fields_autoplaced)
     (property "Reference" "R36" (id 0) (at 389.89 377.5542 90))
-    (property "Value" "470R_0603" (id 1) (at 389.89 384.81 90)
+    (property "Value" "10k_0603" (id 1) (at 389.89 384.81 90)
       (effects (font (size 1.27 1.27)) hide)
     )
@@
     (in_bom yes) (on_board yes) (fields_autoplaced)
     (property "Reference" "R50" (id 0) (at 405.13 288.6542 90))
-    (property "Value" "100k_0603" (id 1) (at 405.13 295.91 90)
+    (property "Value" "10k_0603" (id 1) (at 405.13 295.91 90)
       (effects (font (size 1.27 1.27)) hide)
     )
@@
     (in_bom yes) (on_board yes) (fields_autoplaced)
     (property "Reference" "R39" (id 0) (at 386.08 288.6542 90))
-    (property "Value" "100k_0603" (id 1) (at 386.08 295.91 90)
+    (property "Value" "15k_0603" (id 1) (at 386.08 295.91 90)
       (effects (font (size 1.27 1.27)) hide)
     )
@@
     (in_bom yes) (on_board yes) (fields_autoplaced)
     (property "Reference" "R47" (id 0) (at 405.13 226.4242 90))
-    (property "Value" "100k_0603" (id 1) (at 405.13 233.68 90)
+    (property "Value" "10k_0603" (id 1) (at 405.13 233.68 90)
       (effects (font (size 1.27 1.27)) hide)
     )
@@
     )
     (path "/3774fc9f-9fd2-43d3-8a75-589cc09247b6"
-      (reference "R3") (unit 1) (value "470R_0603") (footprint "4ms_Resistor:R_0603")
+      (reference "R3") (unit 1) (value "10k_0603") (footprint "4ms_Resistor:R_0603")
     )
     (path "/dceacdff-7218-4166-a09c-0285034156d0"
@@
     )
     (path "/365b44b4-ded6-4dbe-a3e5-decae09e3a3f"
-      (reference "R7") (unit 1) (value "470R_0603") (footprint "4ms_Resistor:R_0603")
+      (reference "R7") (unit 1) (value "10k_0603") (footprint "4ms_Resistor:R_0603")
     )
     (path "/d3141b3d-cdaa-4853-9bb6-0e61eeb4071d"
@@
     )
     (path "/975fd9d7-c0ad-4c64-a53b-b51789adb271"
-      (reference "R16") (unit 1) (value "100k_0603") (footprint "4ms_Resistor:R_0603")
+      (reference "R16") (unit 1) (value "10k_0603") (footprint "4ms_Resistor:R_0603")
     )
     (path "/77bb906b-3c99-4315-ab7e-38da1fa8a970"
@@
     )
     (path "/797e0386-7470-4b39-8fbf-ed268b7f1b02"
-      (reference "R22") (unit 1) (value "4.7k_0603") (footprint "4ms_Resistor:R_0603")
+      (reference "R22") (unit 1) (value "10k_0603") (footprint "4ms_Resistor:R_0603")
     )
     (path "/8f3c0007-f897-4426-b9c2-a51e34b8b3f3"
@@
     )
     (path "/8c5ff5ed-8279-439d-923c-892ad5c47963"
-      (reference "R30") (unit 1) (value "100k_0603") (footprint "4ms_Resistor:R_0603")
+      (reference "R30") (unit 1) (value "15k_0603") (footprint "4ms_Resistor:R_0603")
     )
     (path "/4a10fbe9-17b4-45b3-bf1d-98f404b69d04"
@@
     )
     (path "/b87cf6a6-5af0-474e-a254-c49543160b9d"
-      (reference "R36") (unit 1) (value "470R_0603") (footprint "4ms_Resistor:R_0603")
+      (reference "R36") (unit 1) (value "10k_0603") (footprint "4ms_Resistor:R_0603")
     )
     (path "/29d17fca-e716-460c-bba9-de3bce25e9bd"
-      (reference "R37") (unit 1) (value "100k_0603") (footprint "4ms_Resistor:R_0603")
+      (reference "R37") (unit 1) (value "15k_0603") (footprint "4ms_Resistor:R_0603")
     )
     (path "/59047adf-7268-4770-860b-190b9159c88b"
@@
     )
     (path "/cb5be06c-ce1e-4c22-8e6b-d5509c81d1e2"
-      (reference "R39") (unit 1) (value "100k_0603") (footprint "4ms_Resistor:R_0603")
+      (reference "R39") (unit 1) (value "15k_0603") (footprint "4ms_Resistor:R_0603")
     )
     (path "/29221296-c524-4b61-b4ec-b289842d0f75"
@@
     )
     (path "/2dfd7f1d-d9ab-4556-adbf-cde073b1dd42"
-      (reference "R43") (unit 1) (value "100R_0603") (footprint "4ms_Resistor:R_0603")
+      (reference "R43") (unit 1) (value "1k_0603") (footprint "4ms_Resistor:R_0603")
     )
     (path "/b14df35d-e4b9-4eec-86ba-8315fbec5beb"
-      (reference "R44") (unit 1) (value "100k_0603") (footprint "4ms_Resistor:R_0603")
+      (reference "R44") (unit 1) (value "10k_0603") (footprint "4ms_Resistor:R_0603")
     )
     (path "/512b3631-9852-498f-b15d-d4fb7c7f2562"
-      (reference "R45") (unit 1) (value "100k_0603") (footprint "4ms_Resistor:R_0603")
+      (reference "R45") (unit 1) (value "10k_0603") (footprint "4ms_Resistor:R_0603")
     )
     (path "/13f08aa7-5cc2-4e72-96ae-94c8713c15dd"
-      (reference "R46") (unit 1) (value "100R_0603") (footprint "4ms_Resistor:R_0603")
+      (reference "R46") (unit 1) (value "1k_0603") (footprint "4ms_Resistor:R_0603")
     )
     (path "/e974d07c-44db-43fc-8446-9fc16af455d9"
-      (reference "R47") (unit 1) (value "100k_0603") (footprint "4ms_Resistor:R_0603")
+      (reference "R47") (unit 1) (value "10k_0603") (footprint "4ms_Resistor:R_0603")
     )
     (path "/509a756a-633e-416e-a5a5-87fb98076f4f"
-      (reference "R48") (unit 1) (value "100k_0603") (footprint "4ms_Resistor:R_0603")
+      (reference "R48") (unit 1) (value "10k_0603") (footprint "4ms_Resistor:R_0603")
     )
     (path "/b4e85bc8-ac65-41f9-be9e-f43e520f6f6b"
-      (reference "R49") (unit 1) (value "100R_0603") (footprint "4ms_Resistor:R_0603")
+      (reference "R49") (unit 1) (value "1k_0603") (footprint "4ms_Resistor:R_0603")
     )
     (path "/c745fcd4-490e-4f9c-87ce-c9fe1dcc2b2a"
-      (reference "R50") (unit 1) (value "100k_0603") (footprint "4ms_Resistor:R_0603")
+      (reference "R50") (unit 1) (value "10k_0603") (footprint "4ms_Resistor:R_0603")
     )
     (path "/d6cdcc92-0877-4607-a3e6-04f5844d86f2"
